File: Barometer-Bmp280/Barometer.kicad_pcb (KiCad board)
At the start: 2 copper layers, 50 x 31 mm, 7 parts, among them U1 BMP280

Commit message: Route sensors, IMU and radio board
Parts:
- added J1: M80-8770405, KiCad:M808770405, F.Cu at (121.4, 73.8)
- moved C1 9.94 mm to (100.0, 75.8)
- moved C2 9.94 mm to (100.0, 77.7)
- moved U1 8.50 mm to (104.9, 76.6)
Routing:
- net +3.3V: track 12.2 -> 32.6 mm
- net /SDA: track 0.00 -> 16.9 mm
- net /SCL: track 0.00 -> 16.3 mm
- net GND: track 2.03 -> 5.81 mm, vias 0 -> 4
- added copper zone on B.Cu, net GND
Other:
- board text added: "SCL"
- board text added: "SDA"
- board text added: "VOLTAGE"

Commit message: Done with most of the boards
Connections:
- J1 pad 1: unconnected-(J1-Pad1) -> GND
Routing:
- net GND: track 5.81 -> 51.0 mm, vias 4 -> 3
- net +3.3V: track 32.6 -> 42.7 mm
Other:
- board text added: "GND"
- board text added: "Vin"
- board text removed: "VOLTAGE"
Changed lines of the file:
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@@
   (net 3 "/SDA")
   (net 4 "/SCL")
-  (net 5 "unconnected-(J1-Pad1)")
-  (net 6 "unconnected-(J1-PadMH1)")
-  (net 7 "unconnected-(J1-PadMH2)")
-  (net 8 "unconnected-(J1-PadMH3)")
-  (net 9 "unconnected-(J1-PadMH4)")
+  (net 5 "unconnected-(J1-PadMH1)")
+  (net 6 "unconnected-(J1-PadMH2)")
+  (net 7 "unconnected-(J1-PadMH3)")
+  (net 8 "unconnected-(J1-PadMH4)")
   (footprint "Capacitor_SMD:C_0402_1005Metric" (layer "F.Cu")
     (at 99.98 75.76 180)
@@
       (stroke (width 0.1) (type solid)) (layer "F.Fab"))
     (pad "1" thru_hole rect (at 0 0 90) (size 1.2 1.2) (drill 0.7) (layers "*.Cu" "*.Mask")
-      (net 5 "unconnected-(J1-Pad1)") (pinfunction "1") (pintype "passive"))
+      (net 2 "GND") (pinfunction "1") (pintype "passive"))
     (pad "2" thru_hole circle (at -2 0 90) (size 1.2 1.2) (drill 0.7) (layers "*.Cu" "*.Mask")
       (net 3 "/SDA") (pinfunction "2") (pintype "passive"))
@@
       (net 1 "+3.3V") (pinfunction "4") (pintype "passive"))
     (pad "MH1" thru_hole circle (at 2.25 -2.375 90) (size 1.478 1.478) (drill 0.95) (layers "*.Cu" "*.Mask")
-      (net 6 "unconnected-(J1-PadMH1)") (pinfunction "MH1") (pintype "passive"))
+      (net 5 "unconnected-(J1-PadMH1)") (pinfunction "MH1") (pintype "passive+no_connect"))
     (pad "MH2" thru_hole circle (at 2.25 2.375 90) (size 1.478 1.478) (drill 0.95) (layers "*.Cu" "*.Mask")
-      (net 7 "unconnected-(J1-PadMH2)") (pinfunction "MH2") (pintype "passive"))
+      (net 6 "unconnected-(J1-PadMH2)") (pinfunction "MH2") (pintype "passive+no_connect"))
     (pad "MH3" thru_hole circle (at -8.25 2.375 90) (size 1.478 1.478) (drill 0.95) (layers "*.Cu" "*.Mask")
-      (net 8 "unconnected-(J1-PadMH3)") (pinfunction "MH3") (pintype "passive"))
+      (net 7 "unconnected-(J1-PadMH3)") (pinfunction "MH3") (pintype "passive+no_connect"))
     (pad "MH4" thru_hole circle (at -8.25 -2.375 90) (size 1.478 1.478) (drill 0.95) (layers "*.Cu" "*.Mask")
-      (net 9 "unconnected-(J1-PadMH4)") (pinfunction "MH4") (pintype "passive"))
+      (net 8 "unconnected-(J1-PadMH4)") (pinfunction "MH4") (pintype "passive+no_connect"))
     (model "M80-8770405.stp"
       (offset (xyz 0 0 0))
@@
   (gr_line (start 87.1 92.9) (end 137.1 92.9)
     (stroke (width 0.1) (type default)) (layer "Edge.Cuts"))
+  (gr_text "GND" (at 112 72.9) (layer "F.SilkS")
+    (effects (font (size 1 1) (thickness 0.15)))
+  )
   (gr_text "SCL" (at 110.4 77.5) (layer "F.SilkS")
     (effects (font (size 1 1) (thickness 0.1)) (justify left bottom))
   )
   (gr_text "SDA" (at 110.5 75) (layer "F.SilkS")
+    (effects (font (size 0.85 1) (thickness 0.1)) (justify left bottom))
+  )
+  (gr_text "Vin" (at 110.6 79.6) (layer "F.SilkS")
     (effects (font (size 1 1) (thickness 0.1)) (justify left bottom))
   )
-  (gr_text "VOLTAGE" (at 108.5 79.6) (layer "F.SilkS")
-    (effects (font (size 1 1) (thickness 0.1)) (justify left bottom))
-  )
+  (segment (start 100.53 77.73) (end 103.9 81.1) (width 0.25) (layer "F.Cu") (net 1))
   (segment (start 105.25 77.4) (end 105.25 77.9) (width 0.25) (layer "F.Cu") (net 1))
+  (segment (start 107.1 79.75) (end 108 79.75) (width 0.25) (layer "F.Cu") (net 1))
   (segment (start 102.7 75.225) (end 100.995 75.225) (width 0.25) (layer "F.Cu") (net 1))
+  (segment (start 100.46 77.73) (end 100.53 77.73) (width 0.25) (layer "F.Cu") (net 1))
   (segment (start 105.725 78.375) (end 102.7875 78.375) (width 0.25) (layer "F.Cu") (net 1))
   (segment (start 104.6 75.8) (end 104.6 75.3) (width 0.25) (layer "F.Cu") (net 1))
+  (segment (start 103.9 81.1) (end 107.7 81.1) (width 0.25) (layer "F.Cu") (net 1))
   (segment (start 104.525 75.225) (end 102.7 75.225) (width 0.25) (layer "F.Cu") (net 1))
   (segment (start 100.46 75.76) (end 100.46 77.73) (width 0.25) (layer "F.Cu") (net 1))
@@
   (segment (start 102.7875 78.375) (end 101.9 77.4875) (width 0.25) (layer "F.Cu") (net 1))
   (segment (start 104.6 75.3) (end 104.525 75.225) (width 0.25) (layer "F.Cu") (net 1))
+  (segment (start 108 79.75) (end 121.425 79.75) (width 0.25) (layer "F.Cu") (net 1))
+  (segment (start 107.7 81.1) (end 108 80.8) (width 0.25) (layer "F.Cu") (net 1))
   (segment (start 105.25 77.9) (end 105.725 78.375) (width 0.25) (layer "F.Cu") (net 1))
+  (segment (start 108 80.8) (end 108 79.75) (width 0.25) (layer "F.Cu") (net 1))
   (segment (start 103.95 77.4) (end 101.9875 77.4) (width 0.25) (layer "F.Cu") (net 1))
-  (segment (start 107.1 79.75) (end 121.425 79.75) (width 0.25) (layer "F.Cu") (net 1))
   (segment (start 101.9 77.4875) (end 101.9 75.3125) (width 0.25) (layer "F.Cu") (net 1))
   (segment (start 104.6 77.4) (end 104.6 76.784568) (width 0.25) (layer "F.Cu") (net 2))
   (segment (start 103.91 75.76) (end 103.95 75.8) (width 0.3) (layer "F.Cu") (net 2))
-  (segment (start 99.44 75.76) (end 98.6 76.6) (width 0.25) (layer "F.Cu") (net 2))
+  (segment (start 102.5 72.5) (end 102.5 73.75) (width 0.25) (layer "F.Cu") (net 2))
+  (segment (start 99.5 75.76) (end 99.5 75.752391) (width 0.25) (layer "F.Cu") (net 2))
+  (segment (start 97.9 76.13) (end 97.9 72.2) (width 0.25) (layer "F.Cu") (net 2))
+  (segment (start 101.502391 73.75) (end 102.5 73.75) (width 0.25) (layer "F.Cu") (net 2))
   (segment (start 103.95 75.8) (end 103.0495 75.8) (width 0.3) (layer "F.Cu") (net 2))
+  (segment (start 102.5 73.75) (end 121.425 73.75) (width 0.25) (layer "F.Cu") (net 2))
+  (segment (start 99.5 75.752391) (end 101.502391 73.75) (width 0.25) (layer "F.Cu") (net 2))
   (segment (start 105.9 77.4) (end 106.8 78.3) (width 0.25) (layer "F.Cu") (net 2))
+  (segment (start 97.9 72.2) (end 102.2 72.2) (width 0.25) (layer "F.Cu") (net 2))
   (segment (start 99.5 77.73) (end 99.5 77.5) (width 0.25) (layer "F.Cu") (net 2))
   (segment (start 103.0495 75.8) (end 102.9 75.9495) (width 0.3) (layer "F.Cu") (net 2))
-  (segment (start 99.5 77.5) (end 98.6 76.6) (width 0.25) (layer "F.Cu") (net 2))
+  (segment (start 102.2 72.2) (end 102.5 72.5) (width 0.25) (layer "F.Cu") (net 2))
   (segment (start 104.6 76.784568) (end 104.600141 76.784427) (width 0.25) (layer "F.Cu") (net 2))
   (segment (start 99.5 75.76) (end 99.44 75.76) (width 0.25) (layer "F.Cu") (net 2))
+  (segment (start 99.5 77.73) (end 97.9 76.13) (width 0.25) (layer "F.Cu") (net 2))
   (via (at 102.9 75.9495) (size 0.8) (drill 0.4) (layers "F.Cu" "B.Cu") (net 2))
-  (via (at 98.6 76.6) (size 0.8) (drill 0.4) (layers "F.Cu" "B.Cu") (net 2))
   (via (at 104.600141 76.784427) (size 0.8) (drill 0.4) (layers "F.Cu" "B.Cu") (net 2))
   (via (at 106.8 78.3) (size 0.8) (drill 0.4) (layers "F.Cu" "B.Cu") (net 2))
+  (segment (start 104.600141 73.800141) (end 104.6 73.8) (width 0.25) (layer "B.Cu") (net 2))
+  (segment (start 109.9 78.3) (end 109.9 73.8) (width 0.25) (layer "B.Cu") (net 2))
+  (segment (start 102.9 75.9495) (end 102.9 73.8) (width 0.3) (layer "B.Cu") (net 2))
+  (segment (start 104.600141 76.784427) (end 104.600141 73.800141) (width 0.25) (layer "B.Cu") (net 2))
+  (segment (start 106.8 78.3) (end 109.9 78.3) (width 0.25) (layer "B.Cu") (net 2))
   (segment (start 105.25 75.3) (end 105.325 75.225) (width 0.25) (layer "F.Cu") (net 3))
   (segment (start 105.25 75.8) (end 105.25 75.3) (width 0.25) (layer "F.Cu") (net 3))

Commit message: Started fixing layouts
Parts:
- added JP1: SolderJumper_3_Open, Jumper:SolderJumper-3_P1.3mm_Open_RoundedPad1.0x1.5mm_NumberLabels, F.Cu at (106.3, 64.2)
- added R1: 1.5k, Resistor_SMD:R_0201_0603Metric_Pad0.64x0.40mm_HandSolder, F.Cu at (104.9, 66.9)
- added R2: 1.5k, Resistor_SMD:R_0201_0603Metric_Pad0.64x0.40mm_HandSolder, F.Cu at (104.9, 68.7)
Connections:
- U1 pad 5: GND -> Net-(JP1-A)
Routing:
- net GND: track 51.0 -> 23.2 mm, vias 3 -> 2
- net /SDA: track 16.9 -> 0.61 mm
- net /SCL: track 16.3 -> 2.69 mm
- net +3.3V: track 42.7 -> 29.3 mm
- net Net-(JP1-A): track 0.00 -> 8.87 mm, vias 0 -> 1

Commit message: LC24 PCBs
Parts:
- removed J1: M80-8770405, KiCad:M808770405
- added J2: M80-8770422, Harwin-M80-8770422:CONN_M80-87704_HRW, F.Cu at (136.3, 82.4)
- H1, H2, H3, H4: footprint MountingHole:MountingHole_3.2mm_M3_ISO7380_Pad_TopBottom -> Mounting_Wuerth:Mounting_Wuerth_WA-SMSI-M1.6_H1mm_9774010633
- moved H4 57.1 mm to (144.0, 95.7)
- moved H3 50.5 mm to (144.0, 75.7)
- moved H1 38.5 mm to (104.0, 95.7)
- moved R1 30.6 mm to (128.4, 86.6), turned to 90 degrees
- moved C2 28.6 mm to (128.4, 80.6), turned to 90 degrees
- moved H2 28.3 mm to (104.0, 75.7)
- moved R2 27.8 mm to (128.4, 83.5), turned to -90 degrees
- moved C1 26.1 mm to (125.7, 80.6), turned to 90 degrees
- moved JP1 22.1 mm to (114.2, 84.9), turned to 90 degrees
- moved U1 16.4 mm to (119.2, 84.6), turned to -90 degrees
Connections:
- JP1 pad 1: Net-(JP1-A) -> GND
- JP1 pad 2: +3.3V -> Net-(JP1-C)
- JP1 pad 3: GND -> +3.3V
- U1 pad 5: Net-(JP1-A) -> Net-(JP1-C)
Routing:
- net +3.3V: track 29.3 -> 52.1 mm
- net /SDA: track 0.61 -> 19.3 mm
- net /SCL: track 2.69 -> 17.1 mm
- net Net-(JP1-A): track 8.87 -> 0.00 mm, vias 1 -> 0
- net GND: track 23.2 -> 15.3 mm
- net Net-(JP1-C): track 0.00 -> 4.47 mm
- added copper zone on F.Cu, net GND
Other:
- board text added: "Barometer"
- board text added: "VDD"
- board text removed: "Vin"
