File: IMU_BMI088/IMU_BMI088.kicad_pcb (KiCad board)
At the start: 2 copper layers, 50 x 31 mm, 7 parts, among them IC1 BMI088

Commit message: Route sensors, IMU and radio board
Parts:
- added J1: M80-8770405, KiCad:M808770405, F.Cu at (114.2, 96.2)
- moved C2 6.51 mm to (107.4, 90.8), turned to 180 degrees
- moved C1 2.23 mm to (110.6, 84.4)
Routing:
- net +3V3: track 0.00 -> 26.6 mm
- net /SCL: track 0.00 -> 9.55 mm
- net /SDA: track 0.00 -> 7.73 mm
- net GND: track 0.00 -> 6.00 mm, vias 0 -> 3
- added copper zone on B.Cu, net GND
Other:
- board text added: "SCL"
- board text added: "SDA"
- board text added: "Voltage"

Commit message: Done with most of the boards
Parts:
- moved IC1 4.40 mm to (109.5, 83.3)
- moved C1 4.40 mm to (110.4, 80.0)
- moved C2 4.40 mm to (107.2, 86.4)
- moved J1 4.40 mm to (114.0, 91.8)
Connections:
- J1 pad 4: unconnected-(J1-Pad4) -> GND
Routing:
- net GND: track 6.00 -> 32.8 mm
Other:
- board text added: "GND"
- board text added: "Vin"
- board text removed: "Voltage"

Commit message: LC24 PCBs
Parts:
- added JP2: SolderJumper_3_Open, Jumper:SolderJumper-3_P1.3mm_Open_RoundedPad1.0x1.5mm_NumberLabels, F.Cu at (103.3, 93.5)
- added JP3: SolderJumper_3_Open, Jumper:SolderJumper-3_P1.3mm_Open_RoundedPad1.0x1.5mm_NumberLabels, F.Cu at (109.8, 93.5)
- added R1: 1.5k, Resistor_SMD:R_0201_0603Metric_Pad0.64x0.40mm_HandSolder, F.Cu at (113.0, 90.5)
- added R2: 1.5k, Resistor_SMD:R_0201_0603Metric_Pad0.64x0.40mm_HandSolder, F.Cu at (113.0, 87.9)
- H1, H2, H3, H4: footprint MountingHole:MountingHole_3.2mm_M3_ISO7380_Pad_TopBottom -> Mounting_Wuerth:Mounting_Wuerth_WA-SMSI-M1.6_H1mm_9774010633
- J1: value M80-8770405 -> M80-8770422; footprint KiCad:M808770405 -> Harwin-M80-8770422:CONN_M80-87704_HRW
- moved C1 11.3 mm to (103.5, 89.0), turned to 180 degrees
- moved J1 7.31 mm to (118.5, 86.1), turned to -90 degrees
- moved IC1 5.52 mm to (108.0, 88.7)
- moved C2 3.88 mm to (103.5, 87.5)
- moved H3 3.79 mm to (90.0, 98.0)
- moved H4 3.65 mm to (90.0, 78.0)
- moved H2 3.26 mm to (130.0, 98.0)
- moved H1 3.10 mm to (130.0, 78.0)
Connections:
- C1 pad 1: +3V3 -> +3.3V
- C2 pad 1: +3V3 -> +3.3V
- H1 pad 1: (no net) -> GND
- H2 pad 1: (no net) -> GND
- H3 pad 1: (no net) -> GND
- H4 pad 1: (no net) -> GND
- IC1 pad 10: GND -> Net-(IC1-SDO2)
- IC1 pad 11: +3V3 -> +3.3V
- IC1 pad 15: GND -> Net-(IC1-SDO1)
- IC1 pad 3: +3V3 -> +3.3V
- IC1 pad 7: +3V3 -> +3.3V
- J1 pad 1: /SCL -> +3.3V
- J1 pad 2: /SDA -> /SCL
- J1 pad 3: +3V3 -> /SDA
Routing:
- net +3.3V: track 0.00 -> 36.9 mm, vias 0 -> 2
- net +3V3: track 26.6 -> 0.00 mm
- net GND: track 32.8 -> 8.00 mm, vias 3 -> 2
- net Net-(IC1-SDO1): track 0.00 -> 5.00 mm
- net Net-(IC1-SDO2): track 0.00 -> 4.00 mm
- net /SDA: track 7.73 -> 9.11 mm
- net /SCL: track 9.55 -> 8.82 mm
- added copper zone on F.Cu, net GND
Other:
- board text added: "VDD"
- board text removed: "Vin"
