File: MAGNETOMETER/MAGNETOMETER.kicad_pcb (KiCad board)
At the start: 2 copper layers, 50 x 31 mm, 6 parts, among them IC1 MMC5603NJ

Commit message: Route sensors, IMU and radio board
Parts:
- added J1: M80-8770405, KiCad:M808770405, F.Cu at (103.4, 68.8)
Routing:
- net GND: track 6.41 -> 19.6 mm, vias 0 -> 1
- net +3V3: track 3.67 -> 13.7 mm
- net /SDA: track 0.00 -> 9.10 mm
- net /SCL: track 0.00 -> 8.47 mm
- added copper zone on B.Cu, net GND
Other:
- board text added: "SCL"
- board text added: "SDA"
- board text added: "Vin"
Changed lines of the file:
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@@
   (net 3 "/SCL")
   (net 4 "/SDA")
+  (net 5 "unconnected-(J1-PadMH1)")
+  (net 6 "unconnected-(J1-PadMH2)")
+  (net 7 "unconnected-(J1-PadMH3)")
+  (net 8 "unconnected-(J1-PadMH4)")
   (footprint "MMC5603NJ:XDCR_MMC5603NJ" (layer "F.Cu")
     (at 94.7 69)
@@
       (net 2 "GND") (pinfunction "1") (pintype "input"))
   )
+  (footprint "KiCad:M808770405" (layer "F.Cu")
+    (at 103.375 68.75 90)
+    (descr "M80-8770405-2")
+    (tags "Connector")
+    (property "Arrow Part Number" "")
+    (property "Arrow Price/Stock" "")
+    (property "Height" "5.56")
+    (property "Manufacturer_Name" "Harwin")
+    (property "Manufacturer_Part_Number" "M80-8770405")
+    (property "Mouser Part Number" "855-M80-8770405")
+    (property "Mouser Price/Stock" "https://www.mouser.co.uk/ProductDetail/Harwin/M80-8770405?qs=3tymCvhQ29ZPq83M%252Bf8kIA%3D%3D")
+    (property "Sheetfile" "MAGNETOMETER.kicad_sch")
+    (property "Sheetname" "")
+    (property "ki_description" "Datamate L-Tek SIL Male Vertical 3mm Throughboard Connector, latched, gold, 4 contacts")
+    (attr through_hole)
+    (fp_text reference "J1" (at -3 0 90) (layer "F.SilkS")
+        (effects (font (size 1.27 1.27) (thickness 0.254)))
+    )
+    (fp_text value "M80-8770405" (at -3 0 90) (layer "F.SilkS") hide
+        (effects (font (size 1.27 1.27) (thickness 0.254)))
+    )
+    (fp_text user "${REFERENCE}" (at -3 0 90) (layer "F.Fab")
+        (effects (font (size 1.27 1.27) (thickness 0.254)))
+    )
+    (fp_line (start -9.05 1.6) (end -9.05 -1.6)
+      (stroke (width 0.2) (type solid)) (layer "F.SilkS"))
+    (fp_line (start 0 -2.9) (end 0 -2.9)
+      (stroke (width 0.1) (type solid)) (layer "F.SilkS"))
+    (fp_line (start 0 -2.8) (end 0 -2.8)
+      (stroke (width 0.1) (type solid)) (layer "F.SilkS"))
+    (fp_line (start 1.2 -1.9) (end -7.2 -1.9)
+      (stroke (width 0.2) (type solid)) (layer "F.SilkS"))
+    (fp_line (start 1.2 2.08) (end -7.2 2.08)
+      (stroke (width 0.2) (type solid)) (layer "F.SilkS"))
+    (fp_line (start 3.05 -1.6) (end 3.05 1.6)
+      (stroke (width 0.2) (type solid)) (layer "F.SilkS"))
+    (fp_arc (start 0 -2.9) (mid 0.05 -2.85) (end 0 -2.8)
+      (stroke (width 0.1) (type solid)) (layer "F.SilkS"))
+    (fp_arc (start 0 -2.8) (mid -0.05 -2.85) (end 0 -2.9)
+      (stroke (width 0.1) (type solid)) (layer "F.SilkS"))
+    (fp_line (start -10.05 -4.114) (end -10.05 4.114)
+      (stroke (width 0.1) (type solid)) (layer "F.CrtYd"))
+    (fp_line (start -10.05 4.114) (end 4.05 4.114)
+      (stroke (width 0.1) (type solid)) (layer "F.CrtYd"))
+    (fp_line (start 4.05 -4.114) (end -10.05 -4.114)
+      (stroke (width 0.1) (type solid)) (layer "F.CrtYd"))
+    (fp_line (start 4.05 4.114) (end 4.05 -4.114)
+      (stroke (width 0.1) (type solid)) (layer "F.CrtYd"))
+    (fp_line (start -9.05 -1.9) (end 3.05 -1.9)
+      (stroke (width 0.1) (type solid)) (layer "F.Fab"))
+    (fp_line (start -9.05 2.08) (end -9.05 -1.9)
+      (stroke (width 0.1) (type solid)) (layer "F.Fab"))
+    (fp_line (start 3.05 -1.9) (end 3.05 2.08)
+      (stroke (width 0.1) (type solid)) (layer "F.Fab"))
+    (fp_line (start 3.05 2.08) (end -9.05 2.08)
+      (stroke (width 0.1) (type solid)) (layer "F.Fab"))
+    (pad "1" thru_hole rect (at 0 0 90) (size 1.2 1.2) (drill 0.7) (layers "*.Cu" "*.Mask")
+      (net 3 "/SCL") (pinfunction "1") (pintype "passive"))
+    (pad "2" thru_hole circle (at -2 0 90) (size 1.2 1.2) (drill 0.7) (layers "*.Cu" "*.Mask")
+      (net 4 "/SDA") (pinfunction "2") (pintype "passive"))
+    (pad "3" thru_hole circle (at -4 0 90) (size 1.2 1.2) (drill 0.7) (layers "*.Cu" "*.Mask")
+      (net 1 "+3V3") (pinfunction "3") (pintype "passive"))
+    (pad "4" thru_hole circle (at -6 0 90) (size 1.2 1.2) (drill 0.7) (layers "*.Cu" "*.Mask")
+      (net 2 "GND") (pinfunction "4") (pintype "passive"))
+    (pad "MH1" thru_hole circle (at 2.25 -2.375 90) (size 1.478 1.478) (drill 0.95) (layers "*.Cu" "*.Mask")
+      (net 5 "unconnected-(J1-PadMH1)") (pinfunction "MH1") (pintype "passive+no_connect"))
+    (pad "MH2" thru_hole circle (at 2.25 2.375 90) (size 1.478 1.478) (drill 0.95) (layers "*.Cu" "*.Mask")
+      (net 6 "unconnected-(J1-PadMH2)") (pinfunction "MH2") (pintype "passive+no_connect"))
+    (pad "MH3" thru_hole circle (at -8.25 2.375 90) (size 1.478 1.478) (drill 0.95) (layers "*.Cu" "*.Mask")
+      (net 7 "unconnected-(J1-PadMH3)") (pinfunction "MH3") (pintype "passive+no_connect"))
+    (pad "MH4" thru_hole circle (at -8.25 -2.375 90) (size 1.478 1.478) (drill 0.95) (layers "*.Cu" "*.Mask")
+      (net 8 "unconnected-(J1-PadMH4)") (pinfunction "MH4") (pintype "passive+no_connect"))
+    (model "M80-8770405.stp"
+      (offset (xyz 0 0 0))
+      (scale (xyz 1 1 1))
+      (rotate (xyz 0 0 0))
+    )
+  )
   (footprint "Capacitor_SMD:C_0603_1608Metric" (layer "F.Cu")
     (at 93.025 72.6 180)
@@
   (gr_line (start 122 55.7) (end 72 55.7)
     (stroke (width 0.1) (type default)) (layer "Edge.Cuts"))
-  (segment (start 93.8 69.9) (end 94.485 69.215) (width 0.2) (layer "F.Cu") (net 1))
-  (segment (start 93.8 72.6) (end 93.8 69.9) (width 0.2) (layer "F.Cu") (net 1))
+  (gr_text "SCL" (at 96.3 68.6) (layer "F.SilkS")
+    (effects (font (size 1 1) (thickness 0.15)) (justify left bottom))
+  )
+  (gr_text "Vin" (at 96.6 72.8) (layer "F.SilkS")
+    (effects (font (size 1 1) (thickness 0.15)) (justify left bottom))
+  )
+  (gr_text "SDA" (at 96.3 70.6) (layer "F.SilkS")
+    (effects (font (size 1 1) (thickness 0.15)) (justify left bottom))
+  )
+  (segment (start 93.8 72.6) (end 94.4 72) (width 0.2) (layer "F.Cu") (net 1))
+  (segment (start 93.8 69.9) (end 93.8 70.8) (width 0.2) (layer "F.Cu") (net 1))
+  (segment (start 102.025 71.4) (end 103.375 72.75) (width 0.2) (layer "F.Cu") (net 1))
+  (segment (start 94.485 69.215) (end 93.8 69.9) (width 0.2) (layer "F.Cu") (net 1))
+  (segment (start 94.4 71.4) (end 102.025 71.4) (width 0.2) (layer "F.Cu") (net 1))
+  (segment (start 94.4 72) (end 94.4 71.4) (width 0.2) (layer "F.Cu") (net 1))
+  (segment (start 93.8 70.8) (end 94.4 71.4) (width 0.2) (layer "F.Cu") (net 1))
+  (segment (start 92.25 72.6) (end 91.1 72.6) (width 0.2) (layer "F.Cu") (net 2))
   (segment (start 92.3 68.8) (end 92.8 68.3) (width 0.2) (layer "F.Cu") (net 2))
   (segment (start 92.25 72.6) (end 92.3 72.55) (width 0.2) (layer "F.Cu") (net 2))
   (segment (start 94 68.3) (end 94.485 68.785) (width 0.2) (layer "F.Cu") (net 2))
   (segment (start 92.3 72.55) (end 92.3 68.8) (width 0.2) (layer "F.Cu") (net 2))
+  (segment (start 94.4 74.75) (end 103.375 74.75) (width 0.2) (layer "F.Cu") (net 2))
+  (segment (start 92.25 72.6) (end 94.4 74.75) (width 0.2) (layer "F.Cu") (net 2))
   (segment (start 92.8 68.3) (end 94 68.3) (width 0.2) (layer "F.Cu") (net 2))
+  (via (at 91.1 72.6) (size 0.7) (drill 0.3) (layers "F.Cu" "B.Cu") (net 2))
+  (segment (start 103.375 68.75) (end 94.95 68.75) (width 0.2) (layer "F.Cu") (net 3))
+  (segment (start 94.95 68.75) (end 94.915 68.785) (width 0.2) (layer "F.Cu") (net 3))
+  (segment (start 96.45 70.75) (end 94.915 69.215) (width 0.2) (layer "F.Cu") (net 4))
+  (segment (start 103.375 70.75) (end 96.45 70.75) (width 0.2) (layer "F.Cu") (net 4))
+  (zone (net 2) (net_name "GND") (layer "B.Cu") (hatch edge 0.5)
+    (connect_pads (clearance 0.5))
+    (min_thickness 0.25) (filled_areas_thickness no)
+    (fill yes (thermal_gap 0.5) (thermal_bridge_width 0.5))
+    (polygon
+      (pts
+        (xy 72 55.7)
+        (xy 72 86.7)
+        (xy 122.1 86.7)
+        (xy 122 55.7)
+      )
+    )
+  )
 )

Commit message: Done with most of the boards
Parts:
- added R1: 2.7K, Resistor_SMD:R_0201_0603Metric, F.Cu at (96.0, 66.4)
- added R2: 2.7K, Resistor_SMD:R_0201_0603Metric, F.Cu at (97.6, 70.0)
Connections:
- IC1 pad A2: /SCL -> Net-(IC1-SCL)
- IC1 pad B2: /SDA -> Net-(IC1-SDA)
Routing:
- net /SCL: track 8.47 -> 16.5 mm
- net /SDA: track 9.10 -> 14.9 mm
- net Net-(IC1-SCL): track 0.00 -> 2.70 mm, vias 0 -> 1
- net Net-(IC1-SDA): track 0.00 -> 2.37 mm, vias 0 -> 1
- net GND: track 19.6 -> 18.4 mm, vias 1 -> 0
Other:
- board text added: "GND"

Commit message: LC24 PCBs
Parts:
- removed J1: M80-8770405, KiCad:M808770405
- added J2: M80-8770422, Harwin-M80-8770422:CONN_M80-87704_HRW, F.Cu at (105.6, 68.8)
- H1, H2, H3, H4: footprint MountingHole:MountingHole_3.2mm_M3_ISO7380_Pad_TopBottom -> Mounting_Wuerth:Mounting_Wuerth_WA-SMSI-M1.6_H1mm_9774010633
- R1, R2: value 2.7K -> 1.5k; footprint Resistor_SMD:R_0201_0603Metric -> Resistor_SMD:R_0201_0603Metric_Pad0.64x0.40mm_HandSolder
- moved R1 7.30 mm to (99.8, 72.6), turned to 90 degrees
- moved H1 3.78 mm to (117.3, 61.3)
- moved H2 3.73 mm to (117.3, 81.3)
- moved H4 3.17 mm to (77.3, 61.3)
- moved H3 3.11 mm to (77.3, 81.3)
- moved R2 2.27 mm to (99.8, 69.6), turned to -90 degrees
- moved C1 1.40 mm to (94.4, 72.5), turned to 0 degrees
- moved IC1 1.20 mm to (93.8, 69.8)
Connections:
- C1 pad 1: +3V3 -> +3.3V
- IC1 pad A2: Net-(IC1-SCL) -> /SCL
- IC1 pad B1: +3V3 -> +3.3V
- IC1 pad B2: Net-(IC1-SDA) -> /SDA
- R1 pad 1: Net-(IC1-SCL) -> +3.3V
- R1 pad 2: /SCL -> /SDA
- R2 pad 1: Net-(IC1-SDA) -> +3.3V
- R2 pad 2: /SDA -> /SCL
Routing:
- net +3.3V: track 0.00 -> 30.7 mm
- net +3V3: track 13.7 -> 0.00 mm
- net GND: track 18.4 -> 8.94 mm, vias 0 -> 4
- net /SCL: track 16.5 -> 12.6 mm
- net Net-(IC1-SCL): track 2.70 -> 0.00 mm, vias 1 -> 0
- net Net-(IC1-SDA): track 2.37 -> 0.00 mm, vias 1 -> 0
- net /SDA: track 14.9 -> 12.7 mm
- added copper zone on F.Cu, net GND
Other:
- board text added: "Magnetometer"
- board text added: "VDD"
- board text removed: "Vin"
