File: Radio_LoRa/Radio_LoRa.kicad_pcb (KiCad board)
At the start: 2 copper layers, 50 x 31 mm, 6 parts, among them J1 SMA-J-P-H-ST-EM1, U1 RFM95W-915S2

Commit message: Route sensors, IMU and radio board
Parts:
- added J2: M80-8770405, KiCad:M808770405, F.Cu at (117.8, 89.8)
Routing:
- net GND: track 0.00 -> 15.8 mm, vias 0 -> 4
- net /SCK: track 0.00 -> 12.5 mm
- net /MOSI: track 0.00 -> 12.5 mm
- net /MISO: track 0.00 -> 12.5 mm
- net Net-(U1-ANT): track 0.00 -> 10.4 mm
- added copper zone on B.Cu, net GND
Other:
- board text added: "MISO"
- board text added: "MOSI"
- board text added: "SCK"
Changed lines of the file:
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@@
   (net 13 "unconnected-(U1-DIO1-Pad15)")
   (net 14 "unconnected-(U1-DIO2-Pad16)")
+  (net 15 "unconnected-(J2-PadMH1)")
+  (net 16 "unconnected-(J2-PadMH2)")
+  (net 17 "unconnected-(J2-PadMH3)")
+  (net 18 "unconnected-(J2-PadMH4)")
   (footprint "MountingHole:MountingHole_3.2mm_M3_ISO7380_Pad_TopBottom" (layer "F.Cu")
     (at 153 105.3)
@@
     (pad "1" connect circle (at 0 0) (size 5.7 5.7) (layers "B.Cu" "B.Mask")
       (pinfunction "1") (pintype "input"))
+  )
+  (footprint "KiCad:M808770405" (layer "F.Cu")
+    (at 117.775 89.85 90)
+    (descr "M80-8770405-2")
+    (tags "Connector")
+    (property "Arrow Part Number" "")
+    (property "Arrow Price/Stock" "")
+    (property "Height" "5.56")
+    (property "Manufacturer_Name" "Harwin")
+    (property "Manufacturer_Part_Number" "M80-8770405")
+    (property "Mouser Part Number" "855-M80-8770405")
+    (property "Mouser Price/Stock" "https://www.mouser.co.uk/ProductDetail/Harwin/M80-8770405?qs=3tymCvhQ29ZPq83M%252Bf8kIA%3D%3D")
+    (property "Sheetfile" "Radio_LoRa.kicad_sch")
+    (property "Sheetname" "")
+    (property "ki_description" "Datamate L-Tek SIL Male Vertical 3mm Throughboard Connector, latched, gold, 4 contacts")
+    (attr through_hole)
+    (fp_text reference "J2" (at -3 0 90) (layer "F.SilkS")
+        (effects (font (size 1.27 1.27) (thickness 0.254)))
+    )
+    (fp_text value "M80-8770405" (at -3 0 90) (layer "F.SilkS") hide
+        (effects (font (size 1.27 1.27) (thickness 0.254)))
+    )
+    (fp_text user "${REFERENCE}" (at -3 0 90) (layer "F.Fab")
+        (effects (font (size 1.27 1.27) (thickness 0.254)))
+    )
+    (fp_line (start -9.05 1.6) (end -9.05 -1.6)
+      (stroke (width 0.2) (type solid)) (layer "F.SilkS"))
+    (fp_line (start 0 -2.9) (end 0 -2.9)
+      (stroke (width 0.1) (type solid)) (layer "F.SilkS"))
+    (fp_line (start 0 -2.8) (end 0 -2.8)
+      (stroke (width 0.1) (type solid)) (layer "F.SilkS"))
+    (fp_line (start 1.2 -1.9) (end -7.2 -1.9)
+      (stroke (width 0.2) (type solid)) (layer "F.SilkS"))
+    (fp_line (start 1.2 2.08) (end -7.2 2.08)
+      (stroke (width 0.2) (type solid)) (layer "F.SilkS"))
+    (fp_line (start 3.05 -1.6) (end 3.05 1.6)
+      (stroke (width 0.2) (type solid)) (layer "F.SilkS"))
+    (fp_arc (start 0 -2.9) (mid 0.05 -2.85) (end 0 -2.8)
+      (stroke (width 0.1) (type solid)) (layer "F.SilkS"))
+    (fp_arc (start 0 -2.8) (mid -0.05 -2.85) (end 0 -2.9)
+      (stroke (width 0.1) (type solid)) (layer "F.SilkS"))
+    (fp_line (start -10.05 -4.114) (end -10.05 4.114)
+      (stroke (width 0.1) (type solid)) (layer "F.CrtYd"))
+    (fp_line (start -10.05 4.114) (end 4.05 4.114)
+      (stroke (width 0.1) (type solid)) (layer "F.CrtYd"))
+    (fp_line (start 4.05 -4.114) (end -10.05 -4.114)
+      (stroke (width 0.1) (type solid)) (layer "F.CrtYd"))
+    (fp_line (start 4.05 4.114) (end 4.05 -4.114)
+      (stroke (width 0.1) (type solid)) (layer "F.CrtYd"))
+    (fp_line (start -9.05 -1.9) (end 3.05 -1.9)
+      (stroke (width 0.1) (type solid)) (layer "F.Fab"))
+    (fp_line (start -9.05 2.08) (end -9.05 -1.9)
+      (stroke (width 0.1) (type solid)) (layer "F.Fab"))
+    (fp_line (start 3.05 -1.9) (end 3.05 2.08)
+      (stroke (width 0.1) (type solid)) (layer "F.Fab"))
+    (fp_line (start 3.05 2.08) (end -9.05 2.08)
+      (stroke (width 0.1) (type solid)) (layer "F.Fab"))
+    (pad "1" thru_hole rect (at 0 0 90) (size 1.2 1.2) (drill 0.7) (layers "*.Cu" "*.Mask")
+      (net 6 "/NSS") (pinfunction "1") (pintype "passive"))
+    (pad "2" thru_hole circle (at -2 0 90) (size 1.2 1.2) (drill 0.7) (layers "*.Cu" "*.Mask")
+      (net 3 "/MISO") (pinfunction "2") (pintype "passive"))
+    (pad "3" thru_hole circle (at -4 0 90) (size 1.2 1.2) (drill 0.7) (layers "*.Cu" "*.Mask")
+      (net 4 "/MOSI") (pinfunction "3") (pintype "passive"))
+    (pad "4" thru_hole circle (at -6 0 90) (size 1.2 1.2) (drill 0.7) (layers "*.Cu" "*.Mask")
+      (net 5 "/SCK") (pinfunction "4") (pintype "passive"))
+    (pad "MH1" thru_hole circle (at 2.25 -2.375 90) (size 1.478 1.478) (drill 0.95) (layers "*.Cu" "*.Mask")
+      (net 15 "unconnected-(J2-PadMH1)") (pinfunction "MH1") (pintype "passive"))
+    (pad "MH2" thru_hole circle (at 2.25 2.375 90) (size 1.478 1.478) (drill 0.95) (layers "*.Cu" "*.Mask")
+      (net 16 "unconnected-(J2-PadMH2)") (pinfunction "MH2") (pintype "passive"))
+    (pad "MH3" thru_hole circle (at -8.25 2.375 90) (size 1.478 1.478) (drill 0.95) (layers "*.Cu" "*.Mask")
+      (net 17 "unconnected-(J2-PadMH3)") (pinfunction "MH3") (pintype "passive"))
+    (pad "MH4" thru_hole circle (at -8.25 -2.375 90) (size 1.478 1.478) (drill 0.95) (layers "*.Cu" "*.Mask")
+      (net 18 "unconnected-(J2-PadMH4)") (pinfunction "MH4") (pintype "passive"))
+    (model "M80-8770405.stp"
+      (offset (xyz 0 0 0))
+      (scale (xyz 1 1 1))
+      (rotate (xyz 0 0 0))
+    )
   )
   (footprint "RFM95W-915S2:XCVR_RFM95W-915S2" (layer "F.Cu")
@@
   (gr_line (start 111.1 109.3) (end 161.1 109.3)
     (stroke (width 0.1) (type default)) (layer "Edge.Cuts"))
+  (gr_text "MISO" (at 123.3 85.7) (layer "F.SilkS")
+    (effects (font (size 0.7 0.7) (thickness 0.175) bold) (justify left bottom))
+  )
+  (gr_text "MOSI" (at 123.3 87.6) (layer "F.SilkS")
+    (effects (font (size 0.7 0.7) (thickness 0.175) bold) (justify left bottom))
+  )
+  (gr_text "SCK" (at 123.4 89.7) (layer "F.SilkS")
+    (effects (font (size 0.7 0.7) (thickness 0.175) bold) (justify left bottom))
+  )
+  (segment (start 143.3 98.1) (end 139.8 101.6) (width 0.5) (layer "F.Cu") (net 1))
+  (segment (start 139.8 101.6) (end 139.8 107.0625) (width 0.5) (layer "F.Cu") (net 1))
+  (segment (start 127.9 84.1) (end 130.1 84.1) (width 0.3) (layer "F.Cu") (net 2))
+  (segment (start 143.3 96.1) (end 145.6 96.1) (width 0.3) (layer "F.Cu") (net 2))
+  (segment (start 136.975 104.025) (end 137 104) (width 0.25) (layer "F.Cu") (net 2))
+  (segment (start 142.6 104) (end 142.625 104.025) (width 0.25) (layer "F.Cu") (net 2))
+  (segment (start 136.975 106.8625) (end 136.975 104.025) (width 0.25) (layer "F.Cu") (net 2))
+  (segment (start 142.625 104.025) (end 142.625 106.8625) (width 0.25) (layer "F.Cu") (net 2))
+  (via (at 130.1 84.1) (size 0.7) (drill 0.3) (layers "F.Cu" "B.Cu") (net 2))
+  (via (at 137 104) (size 0.8) (drill 0.4) (layers "F.Cu" "B.Cu") (net 2))
+  (via (at 145.6 96.1) (size 0.7) (drill 0.3) (layers "F.Cu" "B.Cu") (net 2))
+  (via (at 142.6 104) (size 0.8) (drill 0.4) (layers "F.Cu" "B.Cu") (net 2))
+  (segment (start 137 104) (end 142.6 104) (width 0.25) (layer "B.Cu") (net 2))
+  (segment (start 117.775 91.85) (end 123.525 86.1) (width 0.5) (layer "F.Cu") (net 3))
+  (segment (start 123.525 86.1) (end 127.9 86.1) (width 0.5) (layer "F.Cu") (net 3))
+  (segment (start 117.775 93.85) (end 123.525 88.1) (width 0.5) (layer "F.Cu") (net 4))
+  (segment (start 123.525 88.1) (end 127.9 88.1) (width 0.5) (layer "F.Cu") (net 4))
+  (segment (start 123.525 90.1) (end 127.9 90.1) (width 0.5) (layer "F.Cu") (net 5))
+  (segment (start 117.775 95.85) (end 123.525 90.1) (width 0.5) (layer "F.Cu") (net 5))
+  (zone (net 2) (net_name "GND") (layer "B.Cu") (hatch edge 0.5)
+    (connect_pads (clearance 0.5))
+    (min_thickness 0.25) (filled_areas_thickness no)
+    (fill yes (thermal_gap 0.5) (thermal_bridge_width 0.5))
+    (polygon
+      (pts
+        (xy 111.1 78.3)
+        (xy 111.1 109.3)
+        (xy 161.1 109.3)
+        (xy 161.1 78.3)
+      )
+    )
+  )
 )

Commit message: Done with most of the boards
Parts:
- added J3: M80-8770405, KiCad:M808770405, F.Cu at (152.2, 90.0)
Connections:
- J2 pad 1: /NSS -> /MISO
- J2 pad 2: /MISO -> /MOSI
- J2 pad 3: /MOSI -> /SCK
- J2 pad 4: /SCK -> /NSS
Routing:
- net /NSS: track 0.00 -> 11.7 mm
- net GND: track 15.8 -> 4.50 mm, vias 4 -> 2
- net /SCK: track 12.5 -> 11.7 mm
- net /MOSI: track 12.5 -> 11.7 mm
Changed lines of the file:
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@@
   (net 17 "unconnected-(J2-PadMH3)")
   (net 18 "unconnected-(J2-PadMH4)")
+  (net 19 "unconnected-(J3-Pad1)")
+  (net 20 "unconnected-(J3-Pad2)")
+  (net 21 "unconnected-(J3-PadMH3)")
+  (net 22 "unconnected-(J3-PadMH4)")
+  (net 23 "unconnected-(J3-PadMH1)")
+  (net 24 "unconnected-(J3-PadMH2)")
   (footprint "MountingHole:MountingHole_3.2mm_M3_ISO7380_Pad_TopBottom" (layer "F.Cu")
     (at 153 105.3)
@@
       (stroke (width 0.1) (type solid)) (layer "F.Fab"))
     (pad "1" thru_hole rect (at 0 0 90) (size 1.2 1.2) (drill 0.7) (layers "*.Cu" "*.Mask")
-      (net 6 "/NSS") (pinfunction "1") (pintype "passive"))
+      (net 3 "/MISO") (pinfunction "1") (pintype "passive"))
     (pad "2" thru_hole circle (at -2 0 90) (size 1.2 1.2) (drill 0.7) (layers "*.Cu" "*.Mask")
-      (net 3 "/MISO") (pinfunction "2") (pintype "passive"))
+      (net 4 "/MOSI") (pinfunction "2") (pintype "passive"))
     (pad "3" thru_hole circle (at -4 0 90) (size 1.2 1.2) (drill 0.7) (layers "*.Cu" "*.Mask")
-      (net 4 "/MOSI") (pinfunction "3") (pintype "passive"))
+      (net 5 "/SCK") (pinfunction "3") (pintype "passive"))
     (pad "4" thru_hole circle (at -6 0 90) (size 1.2 1.2) (drill 0.7) (layers "*.Cu" "*.Mask")
-      (net 5 "/SCK") (pinfunction "4") (pintype "passive"))
+      (net 6 "/NSS") (pinfunction "4") (pintype "passive"))
     (pad "MH1" thru_hole circle (at 2.25 -2.375 90) (size 1.478 1.478) (drill 0.95) (layers "*.Cu" "*.Mask")
-      (net 15 "unconnected-(J2-PadMH1)") (pinfunction "MH1") (pintype "passive"))
+      (net 15 "unconnected-(J2-PadMH1)") (pinfunction "MH1") (pintype "passive+no_connect"))
     (pad "MH2" thru_hole circle (at 2.25 2.375 90) (size 1.478 1.478) (drill 0.95) (layers "*.Cu" "*.Mask")
-      (net 16 "unconnected-(J2-PadMH2)") (pinfunction "MH2") (pintype "passive"))
+      (net 16 "unconnected-(J2-PadMH2)") (pinfunction "MH2") (pintype "passive+no_connect"))
     (pad "MH3" thru_hole circle (at -8.25 2.375 90) (size 1.478 1.478) (drill 0.95) (layers "*.Cu" "*.Mask")
-      (net 17 "unconnected-(J2-PadMH3)") (pinfunction "MH3") (pintype "passive"))
+      (net 17 "unconnected-(J2-PadMH3)") (pinfunction "MH3") (pintype "passive+no_connect"))
     (pad "MH4" thru_hole circle (at -8.25 -2.375 90) (size 1.478 1.478) (drill 0.95) (layers "*.Cu" "*.Mask")
-      (net 18 "unconnected-(J2-PadMH4)") (pinfunction "MH4") (pintype "passive"))
+      (net 18 "unconnected-(J2-PadMH4)") (pinfunction "MH4") (pintype "passive+no_connect"))
     (model "M80-8770405.stp"
       (offset (xyz 0 0 0))
@@
       (pinfunction "1") (pintype "input"))
   )
+  (footprint "KiCad:M808770405" (layer "F.Cu")
+    (at 152.225 89.95 90)
+    (descr "M80-8770405-2")
+    (tags "Connector")
+    (property "Arrow Part Number" "")
+    (property "Arrow Price/Stock" "")
+    (property "Height" "5.56")
+    (property "Manufacturer_Name" "Harwin")
+    (property "Manufacturer_Part_Number" "M80-8770405")
+    (property "Mouser Part Number" "855-M80-8770405")
+    (property "Mouser Price/Stock" "https://www.mouser.co.uk/ProductDetail/Harwin/M80-8770405?qs=3tymCvhQ29ZPq83M%252Bf8kIA%3D%3D")
+    (property "Sheetfile" "Radio_LoRa.kicad_sch")
+    (property "Sheetname" "")
+    (property "ki_description" "Datamate L-Tek SIL Male Vertical 3mm Throughboard Connector, latched, gold, 4 contacts")
+    (attr through_hole)
+    (fp_text reference "J3" (at -3 0 90) (layer "F.SilkS")
+        (effects (font (size 1.27 1.27) (thickness 0.254)))
+    )
+    (fp_text value "M80-8770405" (at -3 0 90) (layer "F.SilkS") hide
+        (effects (font (size 1.27 1.27) (thickness 0.254)))
+    )
+    (fp_text user "${REFERENCE}" (at -3 0 90) (layer "F.Fab")
+        (effects (font (size 1.27 1.27) (thickness 0.254)))
+    )
+    (fp_line (start -9.05 1.6) (end -9.05 -1.6)
+      (stroke (width 0.2) (type solid)) (layer "F.SilkS"))
+    (fp_line (start 0 -2.9) (end 0 -2.9)
+      (stroke (width 0.1) (type solid)) (layer "F.SilkS"))
+    (fp_line (start 0 -2.8) (end 0 -2.8)
+      (stroke (width 0.1) (type solid)) (layer "F.SilkS"))
+    (fp_line (start 1.2 -1.9) (end -7.2 -1.9)
+      (stroke (width 0.2) (type solid)) (layer "F.SilkS"))
+    (fp_line (start 1.2 2.08) (end -7.2 2.08)
+      (stroke (width 0.2) (type solid)) (layer "F.SilkS"))
+    (fp_line (start 3.05 -1.6) (end 3.05 1.6)
+      (stroke (width 0.2) (type solid)) (layer "F.SilkS"))
+    (fp_arc (start 0 -2.9) (mid 0.05 -2.85) (end 0 -2.8)
+      (stroke (width 0.1) (type solid)) (layer "F.SilkS"))
+    (fp_arc (start 0 -2.8) (mid -0.05 -2.85) (end 0 -2.9)
+      (stroke (width 0.1) (type solid)) (layer "F.SilkS"))
+    (fp_line (start -10.05 -4.114) (end -10.05 4.114)
+      (stroke (width 0.1) (type solid)) (layer "F.CrtYd"))
+    (fp_line (start -10.05 4.114) (end 4.05 4.114)
+      (stroke (width 0.1) (type solid)) (layer "F.CrtYd"))
+    (fp_line (start 4.05 -4.114) (end -10.05 -4.114)
+      (stroke (width 0.1) (type solid)) (layer "F.CrtYd"))
+    (fp_line (start 4.05 4.114) (end 4.05 -4.114)
+      (stroke (width 0.1) (type solid)) (layer "F.CrtYd"))
+    (fp_line (start -9.05 -1.9) (end 3.05 -1.9)
+      (stroke (width 0.1) (type solid)) (layer "F.Fab"))
+    (fp_line (start -9.05 2.08) (end -9.05 -1.9)
+      (stroke (width 0.1) (type solid)) (layer "F.Fab"))
+    (fp_line (start 3.05 -1.9) (end 3.05 2.08)
+      (stroke (width 0.1) (type solid)) (layer "F.Fab"))
+    (fp_line (start 3.05 2.08) (end -9.05 2.08)
+      (stroke (width 0.1) (type solid)) (layer "F.Fab"))
+    (pad "1" thru_hole rect (at 0 0 90) (size 1.2 1.2) (drill 0.7) (layers "*.Cu" "*.Mask")
+      (net 19 "unconnected-(J3-Pad1)") (pinfunction "1") (pintype "passive+no_connect"))
+    (pad "2" thru_hole circle (at -2 0 90) (size 1.2 1.2) (drill 0.7) (layers "*.Cu" "*.Mask")
+      (net 20 "unconnected-(J3-Pad2)") (pinfunction "2") (pintype "passive+no_connect"))
+    (pad "3" thru_hole circle (at -4 0 90) (size 1.2 1.2) (drill 0.7) (layers "*.Cu" "*.Mask")
+      (net 11 "+3.3V") (pinfunction "3") (pintype "passive"))
+    (pad "4" thru_hole circle (at -6 0 90) (size 1.2 1.2) (drill 0.7) (layers "*.Cu" "*.Mask")
+      (net 2 "GND") (pinfunction "4") (pintype "passive"))
+    (pad "MH1" thru_hole circle (at 2.25 -2.375 90) (size 1.478 1.478) (drill 0.95) (layers "*.Cu" "*.Mask")
+      (net 23 "unconnected-(J3-PadMH1)") (pinfunction "MH1") (pintype "passive+no_connect"))
+    (pad "MH2" thru_hole circle (at 2.25 2.375 90) (size 1.478 1.478) (drill 0.95) (layers "*.Cu" "*.Mask")
+      (net 24 "unconnected-(J3-PadMH2)") (pinfunction "MH2") (pintype "passive+no_connect"))
+    (pad "MH3" thru_hole circle (at -8.25 2.375 90) (size 1.478 1.478) (drill 0.95) (layers "*.Cu" "*.Mask")
+      (net 21 "unconnected-(J3-PadMH3)") (pinfunction "MH3") (pintype "passive+no_connect"))
+    (pad "MH4" thru_hole circle (at -8.25 -2.375 90) (size 1.478 1.478) (drill 0.95) (layers "*.Cu" "*.Mask")
+      (net 22 "unconnected-(J3-PadMH4)") (pinfunction "MH4") (pintype "passive+no_connect"))
+    (model "M80-8770405.stp"
+      (offset (xyz 0 0 0))
+      (scale (xyz 1 1 1))
+      (rotate (xyz 0 0 0))
+    )
+  )
   (footprint "MountingHole:MountingHole_3.2mm_M3_ISO7380_Pad_TopBottom" (layer "F.Cu")
     (at 153 82.3)
@@
   (segment (start 127.9 84.1) (end 130.1 84.1) (width 0.3) (layer "F.Cu") (net 2))
   (segment (start 143.3 96.1) (end 145.6 96.1) (width 0.3) (layer "F.Cu") (net 2))
-  (segment (start 136.975 104.025) (end 137 104) (width 0.25) (layer "F.Cu") (net 2))
-  (segment (start 142.6 104) (end 142.625 104.025) (width 0.25) (layer "F.Cu") (net 2))
-  (segment (start 136.975 106.8625) (end 136.975 104.025) (width 0.25) (layer "F.Cu") (net 2))
-  (segment (start 142.625 104.025) (end 142.625 106.8625) (width 0.25) (layer "F.Cu") (net 2))
   (via (at 130.1 84.1) (size 0.7) (drill 0.3) (layers "F.Cu" "B.Cu") (net 2))
-  (via (at 137 104) (size 0.8) (drill 0.4) (layers "F.Cu" "B.Cu") (net 2))
   (via (at 145.6 96.1) (size 0.7) (drill 0.3) (layers "F.Cu" "B.Cu") (net 2))
-  (via (at 142.6 104) (size 0.8) (drill 0.4) (layers "F.Cu" "B.Cu") (net 2))
-  (segment (start 137 104) (end 142.6 104) (width 0.25) (layer "B.Cu") (net 2))
-  (segment (start 117.775 91.85) (end 123.525 86.1) (width 0.5) (layer "F.Cu") (net 3))
-  (segment (start 123.525 86.1) (end 127.9 86.1) (width 0.5) (layer "F.Cu") (net 3))
-  (segment (start 117.775 93.85) (end 123.525 88.1) (width 0.5) (layer "F.Cu") (net 4))
-  (segment (start 123.525 88.1) (end 127.9 88.1) (width 0.5) (layer "F.Cu") (net 4))
-  (segment (start 123.525 90.1) (end 127.9 90.1) (width 0.5) (layer "F.Cu") (net 5))
-  (segment (start 117.775 95.85) (end 123.525 90.1) (width 0.5) (layer "F.Cu") (net 5))
+  (segment (start 119.9685 86.1) (end 117.775 88.2935) (width 0.5) (layer "F.Cu") (net 3))
+  (segment (start 117.775 88.2935) (end 117.775 89.85) (width 0.5) (layer "F.Cu") (net 3))
+  (segment (start 127.9 86.1) (end 119.9685 86.1) (width 0.5) (layer "F.Cu") (net 3))
+  (segment (start 127.9 88.1) (end 121.525 88.1) (width 0.5) (layer "F.Cu") (net 4))
+  (segment (start 121.525 88.1) (end 117.775 91.85) (width 0.5) (layer "F.Cu") (net 4))
+  (segment (start 127.9 90.1) (end 121.525 90.1) (width 0.5) (layer "F.Cu") (net 5))
+  (segment (start 121.525 90.1) (end 117.775 93.85) (width 0.5) (layer "F.Cu") (net 5))
+  (segment (start 127.9 92.1) (end 121.525 92.1) (width 0.5) (layer "F.Cu") (net 6))
+  (segment (start 121.525 92.1) (end 117.775 95.85) (width 0.5) (layer "F.Cu") (net 6))
   (zone (net 2) (net_name "GND") (layer "B.Cu") (hatch edge 0.5)
     (connect_pads (clearance 0.5))

Commit message: LC24 PCBs
Parts:
- removed J3: M80-8770405, KiCad:M808770405
- H1, H2, H3, H4: footprint MountingHole:MountingHole_3.2mm_M3_ISO7380_Pad_TopBottom -> Mounting_Wuerth:Mounting_Wuerth_WA-SMSI-M1.6_H1mm_9774010633
- J2: value M80-8770405 -> M80-8770422; footprint KiCad:M808770405 -> Harwin-M80-8770422:CONN_M80-87704_HRW
- moved J2 16.2 mm to (103.0, 96.4)
Connections:
- H1 pad 1: (no net) -> GND
- H2 pad 1: (no net) -> GND
- H3 pad 1: (no net) -> GND
- H4 pad 1: (no net) -> GND
- J2 pad 1: /MISO -> unconnected-(J2-Pad1)
- J2 pad 2: /MOSI -> unconnected-(J2-Pad2)
- J2 pad 3: /SCK -> unconnected-(J2-Pad3)
- J2 pad 4: /NSS -> unconnected-(J2-Pad4)
Routing:
- net /MISO: track 12.6 -> 0.00 mm
- net /SCK: track 11.7 -> 0.00 mm
- net /NSS: track 11.7 -> 0.00 mm
- net /MOSI: track 11.7 -> 0.00 mm
