File: teensy 4.1/teensy 4.1.kicad_pcb (KiCad board)
At the start: 2 copper layers, 4 parts, among them J1 M80-8770405, J4 M80-8770405, J5 M80-8770405, U1 DEV-16771

Commit message: LC24 PCBs
Parts:
- added C1: 100nF, Capacitor_SMD:C_0201_0603Metric, F.Cu at (93.6, 121.1)
- added C2: 470uF, Capacitor_SMD:C_0201_0603Metric, F.Cu at (160.0, 95.5)
- added C3: 0.1uF, Capacitor_SMD:C_0201_0603Metric, F.Cu at (160.0, 88.3)
- added C4: 0.1uF, Capacitor_SMD:C_0201_0603Metric, F.Cu at (163.1, 72.1)
- added C5: 220uF, Capacitor_SMD:C_0201_0603Metric, F.Cu at (170.4, 79.9)
- added H1: MountingHole_Pad, Mounting_Wuerth:Mounting_Wuerth_WA-SMSI-M1.6_H1mm_9774010633, F.Cu at (131.4, 44.9)
- added H2: MountingHole_Pad, Mounting_Wuerth:Mounting_Wuerth_WA-SMSI-M1.6_H1mm_9774010633, F.Cu at (133.1, 132.2)
- added H3: MountingHole_Pad, Mounting_Wuerth:Mounting_Wuerth_WA-SMSI-M1.6_H1mm_9774010633, F.Cu at (82.7, 77.2)
- added H4: MountingHole_Pad, Mounting_Wuerth:Mounting_Wuerth_WA-SMSI-M1.6_H1mm_9774010633, F.Cu at (172.5, 96.6)
- added J2: Battery_Conn, TerminalBlock:TerminalBlock_Altech_AK300-2_P5.00mm, F.Cu at (163.3, 105.7)
- added J6: Conn_Coaxial, Connector_Coaxial:SMA_Amphenol_132134-10_Vertical, F.Cu at (107.9, 102.7)
- added U3: RFM95W-915S2, footprints:IC16_RFM95W-915S2_RFS-M, F.Cu at (91.3, 95.3)
- added U4: LM7805_TO220, Package_TO_SOT_THT:TO-220-3_Vertical, F.Cu at (158.5, 81.0)
- added U5: MAX31855KASA+T, MAX31855:21-0041B_8_MXM, F.Cu at (93.7, 114.5)
- J1: value M80-8770405 -> M80-8770422; footprint KiCad:M808770405 -> Harwin-M80-8770422:CONN_M80-87704_HRW
- J4: value M80-8770405 -> Thermocouple_Conn; footprint KiCad:M808770405 -> TerminalBlock:TerminalBlock_Altech_AK300-2_P5.00mm
- J5: value M80-8770405 -> Extra_Pins; footprint KiCad:M808770405 -> Connector_PinHeader_1.00mm:PinHeader_1x08_P1.00mm_Vertical_SMD_Pin1Right
- moved J5 88.4 mm to (115.0, 48.4), turned to -90 degrees
- moved J4 40.8 mm to (101.1, 120.0), turned to 0 degrees
- moved U1 38.1 mm to (128.3, 62.7), turned to 180 degrees
- moved J1 31.3 mm to (142.6, 84.3)
Connections:
- J1 pad 1: /SPI_CLK -> +3.3V
- J1 pad 2: /SPI_NSS -> /I2C1_SCL
- J1 pad 3: Net-(U1-MOSI) -> /I2C1_SDA
- J1 pad 4: Net-(U1-MISO) -> GND
- J4 pad 1: unconnected-(J4-Pad1) -> Net-(J4-Pin_1)
- J4 pad 2: /I2C1_SCL -> Net-(J4-Pin_2)
- J5 pad 1: unconnected-(J5-Pad1) -> Net-(J5-Pin_1)
- J5 pad 2: unconnected-(J5-Pad2) -> Net-(J5-Pin_2)
- J5 pad 3: unconnected-(J5-Pad3) -> Net-(J5-Pin_3)
- J5 pad 4: unconnected-(J5-Pad4) -> Net-(J5-Pin_4)
- U1 pad 10: /SPI_NSS -> /CS1
- U1 pad 11: Net-(U1-MOSI) -> /MOSI
- U1 pad 12: Net-(U1-MISO) -> /MISO
- U1 pad 24: /ADC_IN10 -> Net-(J5-Pin_1)
- U1 pad 25: /ADC_IN11 -> Net-(J5-Pin_2)
- U1 pad 26: /ADC_IN12 -> Net-(J5-Pin_3)
- U1 pad 27: /ADC_IN13 -> Net-(J5-Pin_4)
- U1 pad 3.3V_1: unconnected-(U1-3.3V-Pad3.3V_1) -> +3.3V
- U1 pad 3.3V_2: unconnected-(U1-3.3V-Pad3.3V_1) -> +3.3V
- U1 pad 3.3V_3: unconnected-(U1-3.3V-Pad3.3V_1) -> +3.3V
- U1 pad 36: unconnected-(U1-CS2-Pad36) -> /CS2
- U1 pad 37: unconnected-(U1-CS3-Pad37) -> /CS3
- U1 pad 38: /ADC_IN14 -> Net-(J5-Pin_5)
- U1 pad 39: /ADC_IN15 -> Net-(J5-Pin_6)
- U1 pad 40: /ADC_IN16 -> Net-(J5-Pin_7)
- U1 pad 41: /ADC_IN17 -> Net-(J5-Pin_8)
- U1 pad USB_GND1: unconnected-(U1-USB_GND-PadUSB_GND1) -> unconnected-(U1-USB_GND-PadUSB_GND1)_0
Routing:
- net +3.3V: track 0.00 -> 218.4 mm
- net /MISO: track 0.00 -> 104.0 mm
- net /CS1: track 0.00 -> 89.2 mm
- net /SPI_CLK: track 0.00 -> 84.9 mm, vias 0 -> 2
- net /MOSI: track 0.00 -> 72.5 mm
- net GND: track 0.00 -> 61.0 mm, vias 0 -> 5
- net Net-(J5-Pin_8): track 0.00 -> 47.9 mm, vias 0 -> 1
- net /CS2: track 0.00 -> 45.1 mm
- net Net-(J5-Pin_7): track 0.00 -> 44.9 mm, vias 0 -> 1
- net Net-(J5-Pin_6): track 0.00 -> 39.0 mm, vias 0 -> 1
- net Net-(J5-Pin_5): track 0.00 -> 37.2 mm, vias 0 -> 1
- net +5V: track 0.00 -> 27.2 mm
- net Net-(J2-Pin_2): track 0.00 -> 27.1 mm
- net /I2C1_SDA: track 0.00 -> 23.0 mm
- net /I2C1_SCL: track 0.00 -> 20.6 mm
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- added copper zone on F.Cu, net GND
Other:
- board outline added: 101 x 101 mm
- board text added: "GND"
- board text added: "I2C Connector"
- board text added: "Rocket Avionics"
- board text added: "SCL"
- board text added: "SDA"
- board text added: "USST"
- board text added: "VDD"
