File: teensy 4.1/teensy 4.1.kicad_sch (KiCad schematic)
At the start: 4 parts, among them J1 M80-8770405, J4 M80-8770405, J5 M80-8770405, U1 DEV-16771

Commit message: Done with most of the boards
Connections:
- net SPI_CLK: now also J1.1; no longer J1.4
- net SPI_NSS: now also J1.2; no longer J1.1
- net at U1.12 (MISO): now also J1.4; no longer J1.2
Other:
- moved on the sheet: J1
Changed lines of the file:
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@@
   (no_connect (at 173.99 144.78))
   (no_connect (at 173.99 96.52))
-  (wire (pts (xy 173.99 109.22) (xy 189.23 109.22))
-    (stroke (width 0) (type default))
-  )
   (wire (pts (xy 128.27 59.69) (xy 128.27 60.96))
     (stroke (width 0) (type default))
   )
-  (wire (pts (xy 189.23 109.22) (xy 189.23 104.14))
-    (stroke (width 0) (type default))
-  )
-  (wire (pts (xy 173.99 106.68) (xy 186.69 106.68))
-    (stroke (width 0) (type default))
-  )
-  (wire (pts (xy 189.23 104.14) (xy 190.5 104.14))
-    (stroke (width 0) (type default))
-  )
-  (wire (pts (xy 184.15 101.6) (xy 184.15 99.06))
+  (wire (pts (xy 173.99 106.68) (xy 187.96 106.68))
+    (stroke (width 0) (type default))
+  )
+  (wire (pts (xy 184.15 97.79) (xy 196.85 97.79))
+    (stroke (width 0) (type default))
+  )
+  (wire (pts (xy 186.69 101.6) (xy 196.85 101.6))
     (stroke (width 0) (type default))
   )
@@
     (stroke (width 0) (type default))
   )
+  (wire (pts (xy 186.69 109.22) (xy 186.69 101.6))
+    (stroke (width 0) (type default))
+  )
   (wire (pts (xy 173.99 142.24) (xy 177.8 142.24))
     (stroke (width 0) (type default))
   )
+  (wire (pts (xy 184.15 101.6) (xy 184.15 97.79))
+    (stroke (width 0) (type default))
+  )
   (wire (pts (xy 125.73 121.92) (xy 133.35 121.92))
     (stroke (width 0) (type default))
@@
     (stroke (width 0) (type default))
   )
+  (wire (pts (xy 196.85 97.79) (xy 196.85 99.06))
+    (stroke (width 0) (type default))
+  )
   (wire (pts (xy 125.73 124.46) (xy 133.35 124.46))
     (stroke (width 0) (type default))
@@
     (stroke (width 0) (type default))
   )
+  (wire (pts (xy 187.96 96.52) (xy 196.85 96.52))
+    (stroke (width 0) (type default))
+  )
   (wire (pts (xy 133.35 129.54) (xy 124.46 129.54))
     (stroke (width 0) (type default))
   )
-  (wire (pts (xy 186.69 106.68) (xy 186.69 101.6))
-    (stroke (width 0) (type default))
-  )
   (wire (pts (xy 133.35 127) (xy 123.19 127))
     (stroke (width 0) (type default))
@@
     (stroke (width 0) (type default))
   )
+  (wire (pts (xy 173.99 109.22) (xy 186.69 109.22))
+    (stroke (width 0) (type default))
+  )
+  (wire (pts (xy 187.96 104.14) (xy 196.85 104.14))
+    (stroke (width 0) (type default))
+  )
   (wire (pts (xy 128.27 60.96) (xy 133.35 60.96))
     (stroke (width 0) (type default))
   )
+  (wire (pts (xy 187.96 106.68) (xy 187.96 104.14))
+    (stroke (width 0) (type default))
+  )
   (wire (pts (xy 173.99 101.6) (xy 184.15 101.6))
     (stroke (width 0) (type default))
   )
-  (wire (pts (xy 184.15 99.06) (xy 190.5 99.06))
-    (stroke (width 0) (type default))
-  )
   (wire (pts (xy 125.73 116.84) (xy 133.35 116.84))
     (stroke (width 0) (type default))
@@
     (stroke (width 0) (type default))
   )
-  (wire (pts (xy 186.69 101.6) (xy 190.5 101.6))
-    (stroke (width 0) (type default))
-  )
   (rectangle (start 83.82 39.37) (end 220.98 152.4)
     (stroke (width 0) (type default))
@@
     (effects (font (size 1.27 1.27)) (justify left bottom))
   )
-  (label "SPI_CLK" (at 190.5 106.68 0) (fields_autoplaced)
+  (label "SPI_CLK" (at 187.96 96.52 0) (fields_autoplaced)
     (effects (font (size 1.27 1.27)) (justify left bottom))
   )
@@
     )
   )
-  (symbol (lib_id "M80-8770405:M80-8770405") (at 190.5 99.06 0) (unit 1)
+  (symbol (lib_id "M80-8770405:M80-8770405") (at 196.85 96.52 0) (unit 1)
     (in_bom yes) (on_board yes) (dnp no) (fields_autoplaced)
-    (property "Reference" "J1" (at 201.93 91.44 0)
-      (effects (font (size 1.27 1.27)))
-    )
-    (property "Value" "M80-8770405" (at 201.93 93.98 0)
-      (effects (font (size 1.27 1.27)))
-    )
-    (property "Footprint" "M808770405" (at 209.55 193.98 0)
-      (effects (font (size 1.27 1.27)) (justify left top) hide)
-    )
-    (property "Datasheet" "https://cdn.harwin.com/pdfs/M80-877.pdf" (at 209.55 293.98 0)
-      (effects (font (size 1.27 1.27)) (justify left top) hide)
-    )
-    (property "Height" "5.56" (at 209.55 493.98 0)
-      (effects (font (size 1.27 1.27)) (justify left top) hide)
-    )
-    (property "Manufacturer_Name" "Harwin" (at 209.55 593.98 0)
-      (effects (font (size 1.27 1.27)) (justify left top) hide)
-    )
-    (property "Manufacturer_Part_Number" "M80-8770405" (at 209.55 693.98 0)
-      (effects (font (size 1.27 1.27)) (justify left top) hide)
-    )
-    (property "Mouser Part Number" "855-M80-8770405" (at 209.55 793.98 0)
-      (effects (font (size 1.27 1.27)) (justify left top) hide)
-    )
-    (property "Mouser Price/Stock" "https://www.mouser.co.uk/ProductDetail/Harwin/M80-8770405?qs=3tymCvhQ29ZPq83M%252Bf8kIA%3D%3D" (at 209.55 893.98 0)
-      (effects (font (size 1.27 1.27)) (justify left top) hide)
-    )
-    (property "Arrow Part Number" "" (at 209.55 993.98 0)
-      (effects (font (size 1.27 1.27)) (justify left top) hide)
-    )
-    (property "Arrow Price/Stock" "" (at 209.55 1093.98 0)
-      (effects (font (size 1.27 1.27)) (justify left top) hide)
-    )
+    (property "Reference" "J1" (at 208.28 88.9 0)
+      (effects (font (size 1.27 1.27)))
+    )
+    (property "Value" "M80-8770405" (at 208.28 91.44 0)
+      (effects (font (size 1.27 1.27)))
+    )
+    (property "Footprint" "M808770405" (at 215.9 191.44 0)
+      (effects (font (size 1.27 1.27)) (justify left top) hide)
+    )
+    (property "Datasheet" "https://cdn.harwin.com/pdfs/M80-877.pdf" (at 215.9 291.44 0)
+      (effects (font (size 1.27 1.27)) (justify left top) hide)
+    )
+    (property "Height" "5.56" (at 215.9 491.44 0)
+      (effects (font (size 1.27 1.27)) (justify left top) hide)
+    )
+    (property "Manufacturer_Name" "Harwin" (at 215.9 591.44 0)
+      (effects (font (size 1.27 1.27)) (justify left top) hide)
+    )
+    (property "Manufacturer_Part_Number" "M80-8770405" (at 215.9 691.44 0)
+      (effects (font (size 1.27 1.27)) (justify left top) hide)
+    )
+    (property "Mouser Part Number" "855-M80-8770405" (at 215.9 791.44 0)
+      (effects (font (size 1.27 1.27)) (justify left top) hide)
+    )
+    (property "Mouser Price/Stock" "https://www.mouser.co.uk/ProductDetail/Harwin/M80-8770405?qs=3tymCvhQ29ZPq83M%252Bf8kIA%3D%3D" (at 215.9 891.44 0)
+      (effects (font (size 1.27 1.27)) (justify left top) hide)
+    )
+    (property "Arrow Part Number" "" (at 215.9 991.44 0)
+      (effects (font (size 1.27 1.27)) (justify left top) hide)
+    )
+    (property "Arrow Price/Stock" "" (at 215.9 1091.44 0)
+      (effects (font (size 1.27 1.27)) (justify left top) hide)
+    )

Commit message: LC24 PCBs
Parts:
- removed J1, J4, J5: M80-8770405, M808770405, symbol M80-8770405:M80-8770405
- added C1: 100nF, Capacitor_SMD:C_0201_0603Metric, symbol Device:C
- added C2: 470uF, Capacitor_SMD:C_0201_0603Metric, symbol Device:C
- added C3, C4: 0.1uF, Capacitor_SMD:C_0201_0603Metric, symbol Device:C
- added C5: 220uF, Capacitor_SMD:C_0201_0603Metric, symbol Device:C
- added H1, H2, H3, H4: MountingHole_Pad, Mounting_Wuerth:Mounting_Wuerth_WA-SMSI-M1.6_H1mm_9774010633, symbol Mechanical:MountingHole_Pad
- added J1: M80-8770422, Harwin-M80-8770422:CONN_M80-87704_HRW, symbol Harwin-M80-8770422:M80-8770422
- added J2: Battery_Conn, TerminalBlock:TerminalBlock_Altech_AK300-2_P5.00mm, symbol Connector:Screw_Terminal_01x02
- added J4: Thermocouple_Conn, TerminalBlock:TerminalBlock_Altech_AK300-2_P5.00mm, symbol Connector:Screw_Terminal_01x02
- added J5: Extra_Pins, Connector_PinHeader_1.00mm:PinHeader_1x08_P1.00mm_Vertical_SMD_Pin1Right, symbol Connector:Conn_01x08_Male
- added J6: Conn_Coaxial, Connector_Coaxial:SMA_Amphenol_132134-10_Vertical, symbol Connector:Conn_Coaxial
- added U3: RFM95W-915S2, footprints:IC16_RFM95W-915S2_RFS-M, symbol RF_Module:RFM95W-915S2
- added U4: LM7805_TO220, Package_TO_SOT_THT:TO-220-3_Vertical, symbol Regulator_Linear:LM7805_TO220
- added U5: MAX31855KASA+T, MAX31855:21-0041B_8_MXM, symbol 2024-07-03_09-08-40:MAX31855KASA+T
Connections:
- net +5V: now also C4.1, C5.1, U4.3 (VO)
- net GND: now also C1.1, C2.2, C3.2, C4.2, C5.2, H1.1, H2.1, H3.1, H4.1, J1.4, J2.1 (Pin_1), J6.2 (Ext), U3.1 (GND), U3.10 (GND), U3.8 (GND), U4.2 (GND), U5.1 (GND)
- net I2C1_SCL: now also J1.2
- net I2C1_SDA: now also J1.3
- net SPI_CLK: now also U3.4 (SCK), U5.5 (SCK)
- net MOSI: now reaches U1.11 (MOSI)
- net MOSI: now also U3.3 (MOSI)
- net MISO: now reaches U1.12 (MISO)
- net MISO: now also U3.2 (MISO), U5.7 (SO)
- net +3.3V: now reaches U1.3.3V_1 (3.3V), U1.3.3V_2 (3.3V), U1.3.3V_3 (3.3V)
- net +3.3V: now also C1.2, J1.1, U3.13 (3.3V), U5.4 (VCC)
- net CS2: now reaches U1.36 (CS2)
- net CS2: now also U3.5 (NSS)
- net CS3: now reaches U1.37 (CS3)
- net ADC_IN10: no longer names the net of U1.24 (A10)
- net ADC_IN10: now also J5.1 (Pin_1)
- net ADC_IN11: no longer names the net of U1.25 (A11)
- net ADC_IN11: now also J5.2 (Pin_2)
- net ADC_IN12: no longer names the net of U1.26 (A12)
- net ADC_IN12: now also J5.3 (Pin_3)
- net ADC_IN13: no longer names the net of U1.27 (A13)
- net ADC_IN13: now also J5.4 (Pin_4)
- net ADC_IN14: no longer names the net of U1.38 (A14)
- net ADC_IN14: now also J5.5 (Pin_5)
- net ADC_IN15: no longer names the net of U1.39 (A15)
- net ADC_IN15: now also J5.6 (Pin_6)
- net ADC_IN16: no longer names the net of U1.40 (A16)
- net ADC_IN16: now also J5.7 (Pin_7)
- net ADC_IN17: no longer names the net of U1.41 (A17)
- net ADC_IN17: now also J5.8 (Pin_8)
- net SPI_NSS renamed CS1
- net CS1: now also U5.6 (*CS)
- new net: J6.1 (In), U3.9 (ANT)
- new net: C2.1, C3.1, J2.2 (Pin_2), U4.1 (VI)
- new net: J4.1 (Pin_1), U5.3 (T+)
- new net: J4.2 (Pin_2), U5.2 (T-)
- no-connect marks 35 -> 39
Other:
- moved on the sheet: U1
